File: lolly.kicad_pcb (KiCad board)
At the start: 2 copper layers, 500 x 500 mm, 512 parts

Commit message: add v0 schema
Parts:
- added Q1 in1: Conn_01x02_Pin, Connector_JST:JST_PH_B2B-PH-K_1x02_P2.00mm_Vertical, F.Cu at (285.5, 285.0)
- added Q1 out1: Conn_01x02_Pin, Connector_JST:JST_PH_B2B-PH-K_1x02_P2.00mm_Vertical, F.Cu at (287.0, 295.0)
- added Q2 in1: Conn_01x02_Pin, Connector_JST:JST_PH_B2B-PH-K_1x02_P2.00mm_Vertical, F.Cu at (305.0, 277.0)
- added Q2 out1: Conn_01x02_Pin, Connector_JST:JST_PH_B2B-PH-K_1x02_P2.00mm_Vertical, F.Cu at (310.0, 293.0)
- added Q3 in1: Conn_01x02_Pin, Connector_JST:JST_PH_B2B-PH-K_1x02_P2.00mm_Vertical, F.Cu at (307.5, 305.5)
- added Q4 in1: Conn_01x02_Pin, Connector_JST:JST_PH_B2B-PH-K_1x02_P2.00mm_Vertical, F.Cu at (293.5, 315.5)
- added Q4 out1: Conn_01x02_Pin, Connector_JST:JST_PH_B2B-PH-K_1x02_P2.00mm_Vertical, F.Cu at (282.5, 317.5)
- added REF**: MountingHole_3.2mm_M3, MountingHole:MountingHole_3.2mm_M3, F.Cu at (229.0, 320.5)
- added REF**: MountingHole_3.2mm_M3, MountingHole:MountingHole_3.2mm_M3, F.Cu at (132.5, 132.5)
- added REF**: MountingHole_3.2mm_M3, MountingHole:MountingHole_3.2mm_M3, F.Cu at (193.5, 407.0)
- added REF**: MountingHole_3.2mm_M3, MountingHole:MountingHole_3.2mm_M3, F.Cu at (458.0, 141.5)
- added REF**: MountingHole_3.2mm_M3, MountingHole:MountingHole_3.2mm_M3, F.Cu at (462.5, 462.5)
- added REF**: MountingHole_3.2mm_M3, MountingHole:MountingHole_3.2mm_M3, F.Cu at (224.0, 267.5)
- added REF**: MountingHole_3.2mm_M3, MountingHole:MountingHole_3.2mm_M3, F.Cu at (333.0, 375.0)
- added REF**: MountingHole_3.2mm_M3, MountingHole:MountingHole_3.2mm_M3, F.Cu at (282.5, 62.5)
- added REF**: MountingHole_3.2mm_M3, MountingHole:MountingHole_3.2mm_M3, F.Cu at (261.0, 373.5)
- added REF**: MountingHole_3.2mm_M3, MountingHole:MountingHole_3.2mm_M3, F.Cu at (276.5, 219.0)
- added REF**: MountingHole_3.2mm_M3, MountingHole:MountingHole_3.2mm_M3, F.Cu at (364.0, 267.5)
- added REF**: MountingHole_3.2mm_M3, MountingHole:MountingHole_3.2mm_M3, F.Cu at (282.5, 537.5)
- added REF**: MountingHole_3.2mm_M3, MountingHole:MountingHole_3.2mm_M3, F.Cu at (338.0, 215.5)
- added REF**: MountingHole_3.2mm_M3, MountingHole:MountingHole_3.2mm_M3, F.Cu at (415.5, 415.5)
- added REF**: MountingHole_3.2mm_M3, MountingHole:MountingHole_3.2mm_M3, F.Cu at (423.5, 176.5)
- added REF**: MountingHole_3.2mm_M3, MountingHole:MountingHole_3.2mm_M3, F.Cu at (370.5, 347.5)
- added REF**: MountingHole_3.2mm_M3_DIN965, MountingHole:MountingHole_3.2mm_M3_DIN965, F.Cu at (537.5, 332.5)
- added REF**: MountingHole_3.2mm_M3, MountingHole:MountingHole_3.2mm_M3, F.Cu at (132.5, 467.5)
- added REF**: MountingHole_3.2mm_M3, MountingHole:MountingHole_3.2mm_M3, F.Cu at (62.5, 267.5)
- added REF**: MountingHole_3.2mm_M3, MountingHole:MountingHole_3.2mm_M3, F.Cu at (537.5, 267.5)
- added REF**: MountingHole_3.2mm_M3, MountingHole:MountingHole_3.2mm_M3, F.Cu at (317.5, 62.5)
- added REF**: MountingHole_3.2mm_M3, MountingHole:MountingHole_3.2mm_M3, F.Cu at (317.5, 537.5)
- added REF**: MountingHole_3.2mm_M3, MountingHole:MountingHole_3.2mm_M3, F.Cu at (62.5, 332.5)
- added VCC - GND: SolderWire-1.5sqmm_1x02_P6mm_D1.7mm_OD3mm, Connector_Wire:SolderWire-1.5sqmm_1x02_P6mm_D1.7mm_OD3mm, F.Cu at (296.5, 545.5)
- added VCC - GND: SolderWire-1.5sqmm_1x02_P6mm_D1.7mm_OD3mm, Connector_Wire:SolderWire-1.5sqmm_1x02_P6mm_D1.7mm_OD3mm, F.Cu at (303.0, 59.5)
- added VCC - GND: SolderWire-1.5sqmm_1x02_P6mm_D1.7mm_OD3mm, Connector_Wire:SolderWire-1.5sqmm_1x02_P6mm_D1.7mm_OD3mm, F.Cu at (319.5, 335.5)
- added VCC - GND: SolderWire-1.5sqmm_1x02_P6mm_D1.7mm_OD3mm, Connector_Wire:SolderWire-1.5sqmm_1x02_P6mm_D1.7mm_OD3mm, F.Cu at (536.5, 296.5)
- added VCC - GND: SolderWire-1.5sqmm_1x02_P6mm_D1.7mm_OD3mm, Connector_Wire:SolderWire-1.5sqmm_1x02_P6mm_D1.7mm_OD3mm, F.Cu at (322.0, 297.0)
- added VCC - GND: SolderWire-1.5sqmm_1x02_P6mm_D1.7mm_OD3mm, Connector_Wire:SolderWire-1.5sqmm_1x02_P6mm_D1.7mm_OD3mm, F.Cu at (537.0, 306.5)
- added VCC - GND: SolderWire-1.5sqmm_1x02_P6mm_D1.7mm_OD3mm, Connector_Wire:SolderWire-1.5sqmm_1x02_P6mm_D1.7mm_OD3mm, F.Cu at (310.0, 63.0)
- added VCC - GND: SolderWire-1.5sqmm_1x02_P6mm_D1.7mm_OD3mm, Connector_Wire:SolderWire-1.5sqmm_1x02_P6mm_D1.7mm_OD3mm, F.Cu at (58.0, 297.5)
- added VCC - GND: SolderWire-1.5sqmm_1x02_P6mm_D1.7mm_OD3mm, Connector_Wire:SolderWire-1.5sqmm_1x02_P6mm_D1.7mm_OD3mm, F.Cu at (255.5, 316.5)
- added VCC - GND: SolderWire-1.5sqmm_1x02_P6mm_D1.7mm_OD3mm, Connector_Wire:SolderWire-1.5sqmm_1x02_P6mm_D1.7mm_OD3mm, F.Cu at (307.5, 545.5)
- added VCC - GND: SolderWire-1.5sqmm_1x02_P6mm_D1.7mm_OD3mm, Connector_Wire:SolderWire-1.5sqmm_1x02_P6mm_D1.7mm_OD3mm, F.Cu at (57.5, 307.0)
- added VCC - GND: SolderWire-1.5sqmm_1x02_P6mm_D1.7mm_OD3mm, Connector_Wire:SolderWire-1.5sqmm_1x02_P6mm_D1.7mm_OD3mm, F.Cu at (279.0, 267.0)
- added q3 out1: Conn_01x02_Pin, Connector_JST:JST_PH_B2B-PH-K_1x02_P2.00mm_Vertical, F.Cu at (319.0, 319.5)
- moved D464 452.0 mm to (377.5, 75.9), turned to 160.92 degrees
- moved D414 445.1 mm to (147.8, 125.6), turned to -138.888 degrees
- moved D469 432.4 mm to (230.3, 100.5), turned to 19.26 degrees
- moved D506 429.2 mm to (249.3, 104.2), turned to -165.468 degrees
- moved D364 427.7 mm to (75.0, 265.3), turned to -98.76 degrees
- moved D511 427.4 mm to (392.5, 90.4), turned to -23.808 degrees
- moved D367 422.0 mm to (111.4, 160.5), turned to 53.508 degrees
- moved D461 420.0 mm to (236.7, 83.9), turned to -163.68 degrees
- moved D503 419.2 mm to (187.7, 153.9), turned to -142.464 degrees
- moved D419 418.1 mm to (148.4, 143.3), turned to 44.052 degrees
- moved D417 416.7 mm to (190.3, 99.7), turned to 28.716 degrees
- moved D411 414.1 mm to (105.7, 205.7), turned to -115.884 degrees
- moved D456 409.3 mm to (138.6, 185.6), turned to -125.34 degrees
- moved D509 407.7 mm to (332.2, 83.6), turned to -8.472 degrees
- moved D474 407.6 mm to (146.4, 202.6), turned to 57.6 degrees
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Connections:
- D1 pad 1: unconnected-(D1-DI-Pad1) -> Net-(D1-DI)
- D1 pad 2: unconnected-(D1-CI-Pad2) -> Net-(D1-CI)
- D107 pad 1: Net-(D106-DO) -> Net-(D107-DI)
- D107 pad 2: Net-(D106-CO) -> Net-(D107-CI)
- D119 pad 1: Net-(D118-DO) -> Net-(D119-DI)
- D119 pad 2: Net-(D118-CO) -> Net-(D119-CI)
- D123 pad 1: Net-(D122-DO) -> Net-(D123-DI)
- D123 pad 2: Net-(D122-CO) -> Net-(D123-CI)
- D128 pad 5: unconnected-(D128-CO-Pad5) -> Net-(D128-CO)
- D128 pad 6: unconnected-(D128-DO-Pad6) -> Net-(D128-DO)
- D129 pad 1: unconnected-(D129-DI-Pad1) -> Net-(D128-DO)
- D129 pad 2: unconnected-(D129-CI-Pad2) -> Net-(D128-CO)
- D129 pad 5: Net-(D129-CO) -> Net-(D119-CI)
- D129 pad 6: Net-(D129-DO) -> Net-(D119-DI)
- D130 pad 1: Net-(D129-DO) -> Net-(D130-DI)
- D130 pad 2: Net-(D129-CO) -> Net-(D130-CI)
- D140 pad 5: Net-(D140-CO) -> Net-(D107-CI)
- D140 pad 6: Net-(D140-DO) -> Net-(D107-DI)
- D141 pad 1: Net-(D140-DO) -> Net-(D141-DI)
- D141 pad 2: Net-(D140-CO) -> Net-(D141-CI)
- D147 pad 1: Net-(D146-DO) -> Net-(D147-DI)
- D147 pad 2: Net-(D146-CO) -> Net-(D147-CI)
- D148 pad 1: Net-(D147-DO) -> Net-(D148-DI)
- D148 pad 2: Net-(D147-CO) -> Net-(D148-CI)
- D150 pad 5: Net-(D150-CO) -> Net-(D141-CI)
- D150 pad 6: Net-(D150-DO) -> Net-(D141-DI)
- D151 pad 1: Net-(D150-DO) -> Net-(D151-DI)
- D151 pad 2: Net-(D150-CO) -> Net-(D151-CI)
- D162 pad 5: Net-(D162-CO) -> Net-(D130-CI)
- D162 pad 6: Net-(D162-DO) -> Net-(D130-DI)
- D163 pad 1: Net-(D162-DO) -> Net-(D163-DI)
- D163 pad 2: Net-(D162-CO) -> Net-(D163-CI)
- D171 pad 5: Net-(D171-CO) -> Net-(D123-CI)
- D171 pad 6: Net-(D171-DO) -> Net-(D123-DI)
- D172 pad 1: Net-(D171-DO) -> Net-(D172-DI)
- D172 pad 2: Net-(D171-CO) -> Net-(D172-CI)
- D182 pad 5: Net-(D182-CO) -> Net-(D163-CI)
- D182 pad 6: Net-(D182-DO) -> Net-(D163-DI)
- D183 pad 1: Net-(D182-DO) -> Net-(D183-DI)
- D183 pad 2: Net-(D182-CO) -> Net-(D183-CI)
- D19 pad 1: Net-(D18-DO) -> Net-(D19-DI)
- D19 pad 2: Net-(D18-CO) -> Net-(D19-CI)
- D194 pad 5: Net-(D194-CO) -> Net-(D151-CI)
- D194 pad 6: Net-(D194-DO) -> Net-(D151-DI)
- D195 pad 1: Net-(D194-DO) -> Net-(D147-DO)
- D195 pad 2: Net-(D194-CO) -> Net-(D147-CO)
- D195 pad 5: Net-(D195-CO) -> Net-(D148-CI)
- D195 pad 6: Net-(D195-DO) -> Net-(D148-DI)
- D196 pad 1: Net-(D195-DO) -> Net-(D196-DI)
- D196 pad 2: Net-(D195-CO) -> Net-(D196-CI)
- D197 pad 1: Net-(D196-DO) -> Net-(D197-DI)
- D197 pad 2: Net-(D196-CO) -> Net-(D197-CI)
- D2 pad 1: Net-(D1-DO) -> Net-(D2-DI)
- D2 pad 2: Net-(D1-CO) -> Net-(D2-CI)
- D206 pad 5: Net-(D206-CO) -> Net-(D183-CI)
- D206 pad 6: Net-(D206-DO) -> Net-(D183-DI)
- D207 pad 1: Net-(D206-DO) -> Net-(D207-DI)
- D207 pad 2: Net-(D206-CO) -> Net-(D207-CI)
- D218 pad 5: Net-(D218-CO) -> Net-(D172-CI)
- D218 pad 6: Net-(D218-DO) -> Net-(D172-DI)
- D219 pad 1: Net-(D218-DO) -> Net-(D219-DI)
- D219 pad 2: Net-(D218-CO) -> Net-(D219-CI)
- D221 pad 1: Net-(D220-DO) -> Net-(D221-DI)
- D221 pad 2: Net-(D220-CO) -> Net-(D221-CI)
- D223 pad 5: Net-(D223-CO) -> Net-(D219-CI)
- D223 pad 6: Net-(D223-DO) -> Net-(D219-DI)
- D224 pad 1: Net-(D223-DO) -> Net-(D224-DI)
- D224 pad 2: Net-(D223-CO) -> Net-(D224-CI)
- D235 pad 5: Net-(D235-CO) -> Net-(D207-CI)
- D235 pad 6: Net-(D235-DO) -> Net-(D207-DI)
- D236 pad 1: Net-(D235-DO) -> Net-(D236-DI)
- D236 pad 2: Net-(D235-CO) -> Net-(D236-CI)
- D244 pad 5: Net-(D244-CO) -> Net-(D197-CI)
- D244 pad 6: Net-(D244-DO) -> Net-(D197-DI)
- D245 pad 1: Net-(D244-DO) -> Net-(D245-DI)
- D245 pad 2: Net-(D244-CO) -> Net-(D245-CI)
- D250 pad 5: Net-(D250-CO) -> Net-(D236-CI)
- D250 pad 6: Net-(D250-DO) -> Net-(D236-DI)
- D251 pad 1: Net-(D250-DO) -> Net-(D251-DI)
- D251 pad 2: Net-(D250-CO) -> Net-(D251-CI)
- D256 pad 5: unconnected-(D256-CO-Pad5) -> Net-(D256-CO)
- D256 pad 6: unconnected-(D256-DO-Pad6) -> Net-(D256-DO)
- D257 pad 1: unconnected-(D257-DI-Pad1) -> Net-(D256-DO)
- D257 pad 2: unconnected-(D257-CI-Pad2) -> Net-(D256-CO)
- D26 pad 1: Net-(D25-DO) -> Net-(D26-DI)
- D26 pad 2: Net-(D25-CO) -> Net-(D26-CI)
- D262 pad 5: Net-(D262-CO) -> Net-(D224-CI)
- D262 pad 6: Net-(D262-DO) -> Net-(D224-DI)
- D263 pad 1: Net-(D262-DO) -> Net-(D263-DI)
- D263 pad 2: Net-(D262-CO) -> Net-(D263-CI)
- D268 pad 5: Net-(D268-CO) -> Net-(D221-CI)
- D268 pad 6: Net-(D268-DO) -> Net-(D221-DI)
- D269 pad 1: Net-(D268-DO) -> Net-(D269-DI)
- D269 pad 2: Net-(D268-CO) -> Net-(D269-CI)
- D277 pad 5: Net-(D277-CO) -> Net-(D263-CI)
- D277 pad 6: Net-(D277-DO) -> Net-(D263-DI)
- D278 pad 1: Net-(D277-DO) -> Net-(D278-DI)
- D278 pad 2: Net-(D277-CO) -> Net-(D278-CI)
- D288 pad 5: Net-(D288-CO) -> Net-(D251-CI)
- D288 pad 6: Net-(D288-DO) -> Net-(D251-DI)
- D289 pad 1: Net-(D288-DO) -> Net-(D289-DI)
- D289 pad 2: Net-(D288-CO) -> Net-(D289-CI)
- D292 pad 5: Net-(D292-CO) -> Net-(D245-CI)
- D292 pad 6: Net-(D292-DO) -> Net-(D245-DI)
- D293 pad 1: Net-(D292-DO) -> Net-(D196-DO)
- D293 pad 2: Net-(D292-CO) -> Net-(D196-CO)
- D295 pad 5: Net-(D295-CO) -> Net-(D289-CI)
- D295 pad 6: Net-(D295-DO) -> Net-(D289-DI)
- D296 pad 1: Net-(D295-DO) -> Net-(D296-DI)
- D296 pad 2: Net-(D295-CO) -> Net-(D296-CI)
- D3 pad 1: Net-(D2-DO) -> Net-(D3-DI)
- D3 pad 2: Net-(D2-CO) -> Net-(D3-CI)
- D3 pad 5: Net-(D3-CO) -> Net-(D2-CI)
- D3 pad 6: Net-(D3-DO) -> Net-(D2-DI)
- D307 pad 5: Net-(D307-CO) -> Net-(D278-CI)
- D307 pad 6: Net-(D307-DO) -> Net-(D278-DI)
- D308 pad 1: Net-(D307-DO) -> Net-(D308-DI)
- D308 pad 2: Net-(D307-CO) -> Net-(D308-CI)
- D317 pad 5: Net-(D317-CO) -> Net-(D269-CI)
- D317 pad 6: Net-(D317-DO) -> Net-(D269-DI)
- D318 pad 1: Net-(D317-DO) -> Net-(D318-DI)
- D318 pad 2: Net-(D317-CO) -> Net-(D318-CI)
- D319 pad 1: Net-(D318-DO) -> Net-(D319-DI)
- D319 pad 2: Net-(D318-CO) -> Net-(D319-CI)
- D330 pad 5: Net-(D330-CO) -> Net-(D308-CI)
- D330 pad 6: Net-(D330-DO) -> Net-(D308-DI)
- D331 pad 1: Net-(D330-DO) -> Net-(D331-DI)
- D331 pad 2: Net-(D330-CO) -> Net-(D331-CI)
- D34 pad 5: Net-(D34-CO) -> Net-(D19-CI)
- D34 pad 6: Net-(D34-DO) -> Net-(D19-DI)
- D341 pad 5: Net-(D341-CO) -> Net-(D296-CI)
- D341 pad 6: Net-(D341-DO) -> Net-(D296-DI)
- D342 pad 1: Net-(D341-DO) -> Net-(D342-DI)
- D342 pad 2: Net-(D341-CO) -> Net-(D342-CI)
- D35 pad 1: Net-(D34-DO) -> Net-(D35-DI)
- D35 pad 2: Net-(D34-CO) -> Net-(D35-CI)
- D350 pad 5: Net-(D350-CO) -> Net-(D331-CI)
- D350 pad 6: Net-(D350-DO) -> Net-(D331-DI)
- D351 pad 1: Net-(D350-DO) -> Net-(D351-DI)
- D351 pad 2: Net-(D350-CO) -> Net-(D351-CI)
- D362 pad 5: Net-(D362-CO) -> Net-(D319-CI)
- D362 pad 6: Net-(D362-DO) -> Net-(D319-DI)
- D363 pad 1: Net-(D362-DO) -> Net-(D363-DI)
- D363 pad 2: Net-(D362-CO) -> Net-(D363-CI)
- D363 pad 5: Net-(D363-CO) -> Net-(D318-CI)
- D363 pad 6: Net-(D363-DO) -> Net-(D318-DI)
- D364 pad 1: Net-(D363-DO) -> Net-(D364-DI)
- D364 pad 2: Net-(D363-CO) -> Net-(D364-CI)
- D364 pad 5: Net-(D364-CO) -> Net-(D363-CI)
- D364 pad 6: Net-(D364-DO) -> Net-(D363-DI)
- D365 pad 1: Net-(D364-DO) -> Net-(D365-DI)
- D365 pad 2: Net-(D364-CO) -> Net-(D365-CI)
- D365 pad 5: Net-(D365-CO) -> Net-(D364-CI)
- D365 pad 6: Net-(D365-DO) -> Net-(D364-DI)
- D366 pad 1: Net-(D365-DO) -> Net-(D366-DI)
- D366 pad 2: Net-(D365-CO) -> Net-(D366-CI)
- D366 pad 5: Net-(D366-CO) -> Net-(D365-CI)
- D366 pad 6: Net-(D366-DO) -> Net-(D365-DI)
- D367 pad 1: Net-(D366-DO) -> Net-(D367-DI)
- D367 pad 2: Net-(D366-CO) -> Net-(D367-CI)
- D367 pad 5: Net-(D367-CO) -> Net-(D366-CI)
- D367 pad 6: Net-(D367-DO) -> Net-(D366-DI)
- D368 pad 1: Net-(D367-DO) -> Net-(D368-DI)
- D368 pad 2: Net-(D367-CO) -> Net-(D368-CI)
- D368 pad 5: Net-(D368-CO) -> Net-(D367-CI)
- D368 pad 6: Net-(D368-DO) -> Net-(D367-DI)
- D369 pad 1: Net-(D368-DO) -> Net-(D369-DI)
- D369 pad 2: Net-(D368-CO) -> Net-(D369-CI)
- D369 pad 5: Net-(D369-CO) -> Net-(D368-CI)
- D369 pad 6: Net-(D369-DO) -> Net-(D368-DI)
- D370 pad 1: Net-(D369-DO) -> Net-(D370-DI)
- D370 pad 2: Net-(D369-CO) -> Net-(D370-CI)
- D370 pad 5: Net-(D370-CO) -> Net-(D369-CI)
- D370 pad 6: Net-(D370-DO) -> Net-(D369-DI)
- D371 pad 1: Net-(D370-DO) -> Net-(D371-DI)
- D371 pad 2: Net-(D370-CO) -> Net-(D371-CI)
- D371 pad 5: Net-(D371-CO) -> Net-(D370-CI)
- D371 pad 6: Net-(D371-DO) -> Net-(D370-DI)
- D372 pad 1: Net-(D371-DO) -> Net-(D372-DI)
- D372 pad 2: Net-(D371-CO) -> Net-(D372-CI)
- D383 pad 5: Net-(D383-CO) -> Net-(D351-CI)
- D383 pad 6: Net-(D383-DO) -> Net-(D351-DI)
- D384 pad 1: Net-(D383-DO) -> Net-(D384-DI)
- D384 pad 2: Net-(D383-CO) -> Net-(D384-CI)
- D384 pad 5: unconnected-(D384-CO-Pad5) -> Net-(D384-CO)
- D384 pad 6: unconnected-(D384-DO-Pad6) -> Net-(D384-DO)
- D385 pad 1: unconnected-(D385-DI-Pad1) -> Net-(D384-DO)
- D385 pad 2: unconnected-(D385-CI-Pad2) -> Net-(D384-CO)
- D390 pad 5: Net-(D390-CO) -> Net-(D342-CI)
- D390 pad 6: Net-(D390-DO) -> Net-(D342-DI)
- D391 pad 1: Net-(D390-DO) -> Net-(D391-DI)
- D391 pad 2: Net-(D390-CO) -> Net-(D391-CI)
- D392 pad 1: Net-(D391-DO) -> Net-(D392-DI)
- D392 pad 2: Net-(D391-CO) -> Net-(D392-CI)
- D395 pad 5: Net-(D395-CO) -> Net-(D384-CI)
- D395 pad 6: Net-(D395-DO) -> Net-(D384-DI)
- D396 pad 1: Net-(D395-DO) -> Net-(D396-DI)
- D396 pad 2: Net-(D395-CO) -> Net-(D396-CI)
- D4 pad 1: Net-(D3-DO) -> Net-(D4-DI)
- D4 pad 2: Net-(D3-CO) -> Net-(D4-CI)
- D4 pad 5: Net-(D4-CO) -> Net-(D3-CI)
- D4 pad 6: Net-(D4-DO) -> Net-(D3-DI)
- D407 pad 5: Net-(D407-CO) -> Net-(D372-CI)
- D407 pad 6: Net-(D407-DO) -> Net-(D372-DI)
- D408 pad 1: Net-(D407-DO) -> Net-(D408-DI)
- D408 pad 2: Net-(D407-CO) -> Net-(D408-CI)
- D408 pad 5: Net-(D408-CO) -> Net-(D371-CI)
- D408 pad 6: Net-(D408-DO) -> Net-(D371-DI)
- D409 pad 1: Net-(D408-DO) -> Net-(D409-DI)
- D409 pad 2: Net-(D408-CO) -> Net-(D409-CI)
- D409 pad 5: Net-(D409-CO) -> Net-(D408-CI)
- D409 pad 6: Net-(D409-DO) -> Net-(D408-DI)
- D410 pad 1: Net-(D409-DO) -> Net-(D410-DI)
- D410 pad 2: Net-(D409-CO) -> Net-(D410-CI)
- D410 pad 5: Net-(D410-CO) -> Net-(D409-CI)
- D410 pad 6: Net-(D410-DO) -> Net-(D409-DI)
- D411 pad 1: Net-(D410-DO) -> Net-(D411-DI)
- D411 pad 2: Net-(D410-CO) -> Net-(D411-CI)
- D411 pad 5: Net-(D411-CO) -> Net-(D410-CI)
- D411 pad 6: Net-(D411-DO) -> Net-(D410-DI)
- D412 pad 1: Net-(D411-DO) -> Net-(D412-DI)
- D412 pad 2: Net-(D411-CO) -> Net-(D412-CI)
- D412 pad 5: Net-(D412-CO) -> Net-(D411-CI)
- D412 pad 6: Net-(D412-DO) -> Net-(D411-DI)
- D413 pad 1: Net-(D412-DO) -> Net-(D413-DI)
- D413 pad 2: Net-(D412-CO) -> Net-(D413-CI)
- D413 pad 5: Net-(D413-CO) -> Net-(D412-CI)
- D413 pad 6: Net-(D413-DO) -> Net-(D412-DI)
- D414 pad 1: Net-(D413-DO) -> Net-(D414-DI)
- D414 pad 2: Net-(D413-CO) -> Net-(D414-CI)
- D414 pad 5: Net-(D414-CO) -> Net-(D413-CI)
- D414 pad 6: Net-(D414-DO) -> Net-(D413-DI)
- D415 pad 1: Net-(D414-DO) -> Net-(D415-DI)
- D415 pad 2: Net-(D414-CO) -> Net-(D415-CI)
- D415 pad 5: Net-(D415-CO) -> Net-(D414-CI)
- D415 pad 6: Net-(D415-DO) -> Net-(D414-DI)
- D416 pad 1: Net-(D415-DO) -> Net-(D416-DI)
- D416 pad 2: Net-(D415-CO) -> Net-(D416-CI)
- D416 pad 5: Net-(D416-CO) -> Net-(D415-CI)
- D416 pad 6: Net-(D416-DO) -> Net-(D415-DI)
- D417 pad 1: Net-(D416-DO) -> Net-(D417-DI)
- D417 pad 2: Net-(D416-CO) -> Net-(D417-CI)
- D417 pad 5: Net-(D417-CO) -> Net-(D416-CI)
- D417 pad 6: Net-(D417-DO) -> Net-(D416-DI)
- D418 pad 1: Net-(D417-DO) -> Net-(D418-DI)
- D418 pad 2: Net-(D417-CO) -> Net-(D418-CI)
- D418 pad 5: Net-(D418-CO) -> Net-(D417-CI)
- D418 pad 6: Net-(D418-DO) -> Net-(D417-DI)
- D419 pad 1: Net-(D418-DO) -> Net-(D419-DI)
- D419 pad 2: Net-(D418-CO) -> Net-(D419-CI)
- D419 pad 5: Net-(D419-CO) -> Net-(D418-CI)
- D419 pad 6: Net-(D419-DO) -> Net-(D418-DI)
- D420 pad 1: Net-(D419-DO) -> Net-(D420-DI)
- D420 pad 2: Net-(D419-CO) -> Net-(D420-CI)
- D420 pad 5: Net-(D420-CO) -> Net-(D419-CI)
- D420 pad 6: Net-(D420-DO) -> Net-(D419-DI)
- D421 pad 1: Net-(D420-DO) -> Net-(D421-DI)
- D421 pad 2: Net-(D420-CO) -> Net-(D421-CI)
- D421 pad 5: Net-(D421-CO) -> Net-(D420-CI)
- D421 pad 6: Net-(D421-DO) -> Net-(D420-DI)
- D422 pad 1: Net-(D421-DO) -> Net-(D422-DI)
- D422 pad 2: Net-(D421-CO) -> Net-(D422-CI)
- D422 pad 5: Net-(D422-CO) -> Net-(D421-CI)
- D422 pad 6: Net-(D422-DO) -> Net-(D421-DI)
- D423 pad 1: Net-(D422-DO) -> Net-(D423-DI)
- D423 pad 2: Net-(D422-CO) -> Net-(D423-CI)
- D423 pad 5: Net-(D423-CO) -> Net-(D422-CI)
- D423 pad 6: Net-(D423-DO) -> Net-(D422-DI)
- D424 pad 1: Net-(D423-DO) -> Net-(D424-DI)
- D424 pad 2: Net-(D423-CO) -> Net-(D424-CI)
- D424 pad 5: Net-(D424-CO) -> Net-(D423-CI)
- D424 pad 6: Net-(D424-DO) -> Net-(D423-DI)
- D425 pad 1: Net-(D424-DO) -> Net-(D425-DI)
- D425 pad 2: Net-(D424-CO) -> Net-(D425-CI)
- D425 pad 5: Net-(D425-CO) -> Net-(D424-CI)
- D425 pad 6: Net-(D425-DO) -> Net-(D424-DI)
- D426 pad 1: Net-(D425-DO) -> Net-(D426-DI)
- D426 pad 2: Net-(D425-CO) -> Net-(D426-CI)
- D437 pad 5: Net-(D437-CO) -> Net-(D396-CI)
- D437 pad 6: Net-(D437-DO) -> Net-(D396-DI)
- D438 pad 1: Net-(D437-DO) -> Net-(D438-DI)
- D438 pad 2: Net-(D437-CO) -> Net-(D438-CI)
- D438 pad 5: Net-(D438-CO) -> Net-(D392-CI)
- D438 pad 6: Net-(D438-DO) -> Net-(D392-DI)
- D439 pad 1: Net-(D438-DO) -> Net-(D391-DO)
- D439 pad 2: Net-(D438-CO) -> Net-(D391-CO)
- D440 pad 5: Net-(D440-CO) -> Net-(D438-CI)
- D440 pad 6: Net-(D440-DO) -> Net-(D438-DI)
- D441 pad 1: Net-(D440-DO) -> Net-(D441-DI)
- D441 pad 2: Net-(D440-CO) -> Net-(D441-CI)
- D451 pad 5: Net-(D451-CO) -> Net-(D426-CI)
- D451 pad 6: Net-(D451-DO) -> Net-(D426-DI)
- D452 pad 1: Net-(D451-DO) -> Net-(D452-DI)
- D452 pad 2: Net-(D451-CO) -> Net-(D452-CI)
- D452 pad 5: Net-(D452-CO) -> Net-(D425-CI)
- D452 pad 6: Net-(D452-DO) -> Net-(D425-DI)
- D453 pad 1: Net-(D452-DO) -> Net-(D453-DI)
- D453 pad 2: Net-(D452-CO) -> Net-(D453-CI)
- D453 pad 5: Net-(D453-CO) -> Net-(D452-CI)
- D453 pad 6: Net-(D453-DO) -> Net-(D452-DI)
- D454 pad 1: Net-(D453-DO) -> Net-(D454-DI)
- D454 pad 2: Net-(D453-CO) -> Net-(D454-CI)
- D454 pad 5: Net-(D454-CO) -> Net-(D453-CI)
- D454 pad 6: Net-(D454-DO) -> Net-(D453-DI)
- D455 pad 1: Net-(D454-DO) -> Net-(D455-DI)
- D455 pad 2: Net-(D454-CO) -> Net-(D455-CI)
- D455 pad 5: Net-(D455-CO) -> Net-(D454-CI)
- D455 pad 6: Net-(D455-DO) -> Net-(D454-DI)
- D456 pad 1: Net-(D455-DO) -> Net-(D456-DI)
- D456 pad 2: Net-(D455-CO) -> Net-(D456-CI)
- D456 pad 5: Net-(D456-CO) -> Net-(D455-CI)
- D456 pad 6: Net-(D456-DO) -> Net-(D455-DI)
- D457 pad 1: Net-(D456-DO) -> Net-(D457-DI)
- D457 pad 2: Net-(D456-CO) -> Net-(D457-CI)
- D457 pad 5: Net-(D457-CO) -> Net-(D456-CI)
- D457 pad 6: Net-(D457-DO) -> Net-(D456-DI)
- D458 pad 1: Net-(D457-DO) -> Net-(D458-DI)
- D458 pad 2: Net-(D457-CO) -> Net-(D458-CI)
- D458 pad 5: Net-(D458-CO) -> Net-(D457-CI)
- D458 pad 6: Net-(D458-DO) -> Net-(D457-DI)
- D459 pad 1: Net-(D458-DO) -> Net-(D459-DI)
- D459 pad 2: Net-(D458-CO) -> Net-(D459-CI)
- D459 pad 5: Net-(D459-CO) -> Net-(D458-CI)
- D459 pad 6: Net-(D459-DO) -> Net-(D458-DI)
- D460 pad 1: Net-(D459-DO) -> Net-(D460-DI)
- D460 pad 2: Net-(D459-CO) -> Net-(D460-CI)
- D460 pad 5: Net-(D460-CO) -> Net-(D459-CI)
- D460 pad 6: Net-(D460-DO) -> Net-(D459-DI)
- D461 pad 1: Net-(D460-DO) -> Net-(D461-DI)
- D461 pad 2: Net-(D460-CO) -> Net-(D461-CI)
- D461 pad 5: Net-(D461-CO) -> Net-(D460-CI)
- D461 pad 6: Net-(D461-DO) -> Net-(D460-DI)
- D462 pad 1: Net-(D461-DO) -> Net-(D462-DI)
- D462 pad 2: Net-(D461-CO) -> Net-(D462-CI)
- D462 pad 5: Net-(D462-CO) -> Net-(D461-CI)
- D462 pad 6: Net-(D462-DO) -> Net-(D461-DI)
- D463 pad 1: Net-(D462-DO) -> Net-(D463-DI)
- D463 pad 2: Net-(D462-CO) -> Net-(D463-CI)
- D463 pad 5: Net-(D463-CO) -> Net-(D462-CI)
- D463 pad 6: Net-(D463-DO) -> Net-(D462-DI)
- D464 pad 1: Net-(D463-DO) -> Net-(D25-DO)
- D464 pad 2: Net-(D463-CO) -> Net-(D25-CO)
- D467 pad 1: Net-(D466-DO) -> Net-(D467-DI)
- D467 pad 2: Net-(D466-CO) -> Net-(D467-CI)
- D467 pad 5: Net-(D467-CO) -> Net-(D463-CI)
- D467 pad 6: Net-(D467-DO) -> Net-(D463-DI)
- D468 pad 1: Net-(D467-DO) -> Net-(D468-DI)
- D468 pad 2: Net-(D467-CO) -> Net-(D468-CI)
- D468 pad 5: Net-(D468-CO) -> Net-(D467-CI)
- D468 pad 6: Net-(D468-DO) -> Net-(D467-DI)
- D469 pad 1: Net-(D468-DO) -> Net-(D469-DI)
- D469 pad 2: Net-(D468-CO) -> Net-(D469-CI)
- D469 pad 5: Net-(D469-CO) -> Net-(D468-CI)
- D469 pad 6: Net-(D469-DO) -> Net-(D468-DI)
- D47 pad 1: Net-(D46-DO) -> Net-(D47-DI)
- D47 pad 2: Net-(D46-CO) -> Net-(D47-CI)
- D470 pad 1: Net-(D469-DO) -> Net-(D470-DI)
- D470 pad 2: Net-(D469-CO) -> Net-(D470-CI)
- D470 pad 5: Net-(D470-CO) -> Net-(D469-CI)
- D470 pad 6: Net-(D470-DO) -> Net-(D469-DI)
- D471 pad 1: Net-(D470-DO) -> Net-(D471-DI)
- D471 pad 2: Net-(D470-CO) -> Net-(D471-CI)
- D471 pad 5: Net-(D471-CO) -> Net-(D470-CI)
- D471 pad 6: Net-(D471-DO) -> Net-(D470-DI)
- D472 pad 1: Net-(D471-DO) -> Net-(D472-DI)
- D472 pad 2: Net-(D471-CO) -> Net-(D472-CI)
- D472 pad 5: Net-(D472-CO) -> Net-(D471-CI)
- D472 pad 6: Net-(D472-DO) -> Net-(D471-DI)
- D473 pad 1: Net-(D472-DO) -> Net-(D473-DI)
- D473 pad 2: Net-(D472-CO) -> Net-(D473-CI)
- D473 pad 5: Net-(D473-CO) -> Net-(D472-CI)
- D473 pad 6: Net-(D473-DO) -> Net-(D472-DI)
- D474 pad 1: Net-(D473-DO) -> Net-(D474-DI)
- D474 pad 2: Net-(D473-CO) -> Net-(D474-CI)
- D474 pad 5: Net-(D474-CO) -> Net-(D473-CI)
- D474 pad 6: Net-(D474-DO) -> Net-(D473-DI)
- D475 pad 1: Net-(D474-DO) -> Net-(D475-DI)
- D475 pad 2: Net-(D474-CO) -> Net-(D475-CI)
- D475 pad 5: Net-(D475-CO) -> Net-(D474-CI)
- D475 pad 6: Net-(D475-DO) -> Net-(D474-DI)
- D476 pad 1: Net-(D475-DO) -> Net-(D476-DI)
- D476 pad 2: Net-(D475-CO) -> Net-(D476-CI)
- D476 pad 5: Net-(D476-CO) -> Net-(D475-CI)
- D476 pad 6: Net-(D476-DO) -> Net-(D475-DI)
- D477 pad 1: Net-(D476-DO) -> Net-(D477-DI)
- D477 pad 2: Net-(D476-CO) -> Net-(D477-CI)
- D477 pad 5: Net-(D477-CO) -> Net-(D476-CI)
- D477 pad 6: Net-(D477-DO) -> Net-(D476-DI)
- D478 pad 1: Net-(D477-DO) -> Net-(D478-DI)
- D478 pad 2: Net-(D477-CO) -> Net-(D478-CI)
- D478 pad 5: Net-(D478-CO) -> Net-(D477-CI)
- D478 pad 6: Net-(D478-DO) -> Net-(D477-DI)
- D479 pad 1: Net-(D478-DO) -> Net-(D479-DI)
- D479 pad 2: Net-(D478-CO) -> Net-(D479-CI)
- D48 pad 1: Net-(D47-DO) -> Net-(D48-DI)
- D48 pad 2: Net-(D47-CO) -> Net-(D48-CI)
- D48 pad 5: Net-(D48-CO) -> Net-(D47-CI)
- D48 pad 6: Net-(D48-DO) -> Net-(D47-DI)
- D487 pad 5: Net-(D487-CO) -> Net-(D441-CI)
- D487 pad 6: Net-(D487-DO) -> Net-(D441-DI)
- D488 pad 1: Net-(D487-DO) -> Net-(D2-DO)
- D488 pad 2: Net-(D487-CO) -> Net-(D2-CO)
- D49 pad 1: Net-(D48-DO) -> Net-(D1-DO)
- D49 pad 2: Net-(D48-CO) -> Net-(D1-CO)
- D496 pad 5: Net-(D496-CO) -> Net-(D479-CI)
- D496 pad 6: Net-(D496-DO) -> Net-(D479-DI)
- D497 pad 1: Net-(D496-DO) -> Net-(D497-DI)
- D497 pad 2: Net-(D496-CO) -> Net-(D497-CI)
- D497 pad 5: Net-(D497-CO) -> Net-(D478-CI)
- D497 pad 6: Net-(D497-DO) -> Net-(D478-DI)
- D498 pad 1: Net-(D497-DO) -> Net-(D498-DI)
- D498 pad 2: Net-(D497-CO) -> Net-(D498-CI)
- D498 pad 5: Net-(D498-CO) -> Net-(D497-CI)
- D498 pad 6: Net-(D498-DO) -> Net-(D497-DI)
- D499 pad 1: Net-(D498-DO) -> Net-(D499-DI)
- D499 pad 2: Net-(D498-CO) -> Net-(D499-CI)
- D499 pad 5: Net-(D499-CO) -> Net-(D498-CI)
- D499 pad 6: Net-(D499-DO) -> Net-(D498-DI)
- D5 pad 1: Net-(D4-DO) -> Net-(D5-DI)
- D5 pad 2: Net-(D4-CO) -> Net-(D5-CI)
- D5 pad 5: Net-(D5-CO) -> Net-(D4-CI)
- D5 pad 6: Net-(D5-DO) -> Net-(D4-DI)
- D50 pad 5: Net-(D50-CO) -> Net-(D48-CI)
- D50 pad 6: Net-(D50-DO) -> Net-(D48-DI)
- D500 pad 1: Net-(D499-DO) -> Net-(D500-DI)
- D500 pad 2: Net-(D499-CO) -> Net-(D500-CI)
- D500 pad 5: Net-(D500-CO) -> Net-(D499-CI)
- D500 pad 6: Net-(D500-DO) -> Net-(D499-DI)
- D501 pad 1: Net-(D500-DO) -> Net-(D501-DI)
- D501 pad 2: Net-(D500-CO) -> Net-(D501-CI)
- D501 pad 5: Net-(D501-CO) -> Net-(D500-CI)
- D501 pad 6: Net-(D501-DO) -> Net-(D500-DI)
- D502 pad 1: Net-(D501-DO) -> Net-(D502-DI)
- D502 pad 2: Net-(D501-CO) -> Net-(D502-CI)
- D502 pad 5: Net-(D502-CO) -> Net-(D501-CI)
- D502 pad 6: Net-(D502-DO) -> Net-(D501-DI)
- D503 pad 1: Net-(D502-DO) -> Net-(D503-DI)
- D503 pad 2: Net-(D502-CO) -> Net-(D503-CI)
- D503 pad 5: Net-(D503-CO) -> Net-(D502-CI)
- D503 pad 6: Net-(D503-DO) -> Net-(D502-DI)
- D504 pad 1: Net-(D503-DO) -> Net-(D504-DI)
- D504 pad 2: Net-(D503-CO) -> Net-(D504-CI)
- D504 pad 5: Net-(D504-CO) -> Net-(D503-CI)
- D504 pad 6: Net-(D504-DO) -> Net-(D503-DI)
- D505 pad 1: Net-(D504-DO) -> Net-(D505-DI)
- D505 pad 2: Net-(D504-CO) -> Net-(D505-CI)
- D505 pad 5: Net-(D505-CO) -> Net-(D504-CI)
- D505 pad 6: Net-(D505-DO) -> Net-(D504-DI)
- D506 pad 1: Net-(D505-DO) -> Net-(D506-DI)
- D506 pad 2: Net-(D505-CO) -> Net-(D506-CI)
- D506 pad 5: Net-(D506-CO) -> Net-(D505-CI)
- D506 pad 6: Net-(D506-DO) -> Net-(D505-DI)
- D507 pad 1: Net-(D506-DO) -> Net-(D18-DO)
- D507 pad 2: Net-(D506-CO) -> Net-(D18-CO)
- D507 pad 5: Net-(D507-CO) -> Net-(D506-CI)
- D507 pad 6: Net-(D507-DO) -> Net-(D506-DI)
- D508 pad 1: Net-(D507-DO) -> Net-(D466-DO)
- D508 pad 2: Net-(D507-CO) -> Net-(D466-CO)
- D51 pad 1: Net-(D50-DO) -> Net-(D51-DI)
- D51 pad 2: Net-(D50-CO) -> Net-(D51-CI)
- D512 pad 5: unconnected-(D512-CO-Pad5) -> Net-(D512-CO)
- D512 pad 6: unconnected-(D512-DO-Pad6) -> Net-(D512-DO)
- D6 pad 1: Net-(D5-DO) -> Net-(D47-DO)
- D6 pad 2: Net-(D5-CO) -> Net-(D47-CO)
- D6 pad 5: Net-(D6-CO) -> Net-(D5-CI)
- D6 pad 6: Net-(D6-DO) -> Net-(D5-DI)
- D61 pad 5: Net-(D61-CO) -> Net-(D35-CI)
- D61 pad 6: Net-(D61-DO) -> Net-(D35-DI)
- D62 pad 1: Net-(D61-DO) -> Net-(D62-DI)
- D62 pad 2: Net-(D61-CO) -> Net-(D62-CI)
- D7 pad 1: Net-(D6-DO) -> Net-(D46-DO)
- D7 pad 2: Net-(D6-CO) -> Net-(D46-CO)
- D73 pad 5: Net-(D73-CO) -> Net-(D26-CI)
- D73 pad 6: Net-(D73-DO) -> Net-(D26-DI)
- D74 pad 1: Net-(D73-DO) -> Net-(D122-DO)
- D74 pad 2: Net-(D73-CO) -> Net-(D122-CO)
- D76 pad 1: Net-(D75-DO) -> Net-(D118-DO)
- D76 pad 2: Net-(D75-CO) -> Net-(D118-CO)
- D87 pad 5: Net-(D87-CO) -> Net-(D62-CI)
- D87 pad 6: Net-(D87-DO) -> Net-(D62-DI)
- D88 pad 1: Net-(D87-DO) -> Net-(D106-DO)
- D88 pad 2: Net-(D87-CO) -> Net-(D106-CO)
- D97 pad 5: Net-(D97-CO) -> Net-(D51-CI)
- D97 pad 6: Net-(D97-DO) -> Net-(D51-DI)
- D98 pad 1: Net-(D97-DO) -> Net-(D146-DO)
- D98 pad 2: Net-(D97-CO) -> Net-(D146-CO)
Routing:
- net GND: track 0.00 -> 1202.5 mm, vias 0 -> 519
- net Net-(D512-DO): track 0.00 -> 256.9 mm, vias 0 -> 1
- net Net-(D512-CO): track 0.00 -> 242.8 mm, vias 0 -> 1
- net Net-(D318-CO): track 0.00 -> 237.6 mm, vias 0 -> 1
- net Net-(D220-DO): track 0.00 -> 232.8 mm, vias 0 -> 1
- net Net-(D220-CO): track 0.00 -> 230.0 mm, vias 0 -> 1
- net Net-(D318-DO): track 0.00 -> 225.5 mm, vias 0 -> 1
- net Net-(D75-DO): track 0.00 -> 218.0 mm, vias 0 -> 1
- net Net-(D75-CO): track 0.00 -> 212.9 mm, vias 0 -> 1
- net Net-(D25-CO): track 0.00 -> 154.0 mm
- net Net-(D25-DO): track 0.00 -> 149.8 mm
- net Net-(D26-CI): track 0.00 -> 105.9 mm
- net Net-(D26-DI): track 0.00 -> 100.7 mm
- net Net-(D221-CI): track 0.00 -> 97.6 mm
- net Net-(D123-CI): track 0.00 -> 95.7 mm
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Other:
- outline, holes or cut-outs redrawn
