File: lolly.kicad_sch (KiCad schematic)
At the start: 512 parts

Commit message: add v0 schema
Parts:
- added Q1 in1: Conn_01x02_Pin, Connector_JST:JST_PH_B2B-PH-K_1x02_P2.00mm_Vertical, symbol Connector:Conn_01x02_Pin
- added Q1 out1: Conn_01x02_Pin, Connector_JST:JST_PH_B2B-PH-K_1x02_P2.00mm_Vertical, symbol Connector:Conn_01x02_Pin
- added Q2 in1: Conn_01x02_Pin, Connector_JST:JST_PH_B2B-PH-K_1x02_P2.00mm_Vertical, symbol Connector:Conn_01x02_Pin
- added Q2 out1: Conn_01x02_Pin, Connector_JST:JST_PH_B2B-PH-K_1x02_P2.00mm_Vertical, symbol Connector:Conn_01x02_Pin
- added Q3 in1: Conn_01x02_Pin, Connector_JST:JST_PH_B2B-PH-K_1x02_P2.00mm_Vertical, symbol Connector:Conn_01x02_Pin
- added Q4 in1: Conn_01x02_Pin, Connector_JST:JST_PH_B2B-PH-K_1x02_P2.00mm_Vertical, symbol Connector:Conn_01x02_Pin
- added Q4 out1: Conn_01x02_Pin, Connector_JST:JST_PH_B2B-PH-K_1x02_P2.00mm_Vertical, symbol Connector:Conn_01x02_Pin
- added q3 out1: Conn_01x02_Pin, Connector_JST:JST_PH_B2B-PH-K_1x02_P2.00mm_Vertical, symbol Connector:Conn_01x02_Pin
Connections:
- net at D106.5 (CO): now also D88.2 (CI); no longer D107.2 (CI)
- net at D106.6 (DO): now also D88.1 (DI); no longer D107.1 (DI)
- net at D498.1 (DI): now also D499.6 (DO); no longer D497.6 (DO)
- net at D498.2 (CI): now also D499.5 (CO); no longer D497.5 (CO)
- net at D499.2 (CI): now also D500.5 (CO); no longer D498.5 (CO)
- net at D499.1 (DI): now also D500.6 (DO); no longer D498.6 (DO)
- net at D363.6 (DO): now also D318.1 (DI); no longer D364.1 (DI)
- net at D363.5 (CO): now also D318.2 (CI); no longer D364.2 (CI)
- net at D364.5 (CO): now also D363.2 (CI); no longer D365.2 (CI)
- net at D364.6 (DO): now also D363.1 (DI); no longer D365.1 (DI)
- net at D477.6 (DO): now also D476.1 (DI); no longer D478.1 (DI)
- net at D477.5 (CO): now also D476.2 (CI); no longer D478.2 (CI)
- net at D479.2 (CI): now also D496.5 (CO); no longer D478.5 (CO)
- net at D479.1 (DI): now also D496.6 (DO); no longer D478.6 (DO)
- net at D384.1 (DI): now also D395.6 (DO); no longer D383.6 (DO)
- net at D384.2 (CI): now also D395.5 (CO); no longer D383.5 (CO)
- net at D384.5 (CO): now also D385.2 (CI)
- net at D384.6 (DO): now also D385.1 (DI)
- net at D51.2 (CI): now also D97.5 (CO); no longer D50.5 (CO)
- net at D51.1 (DI): now also D97.6 (DO); no longer D50.6 (DO)
- net at D455.1 (DI): now also D456.6 (DO); no longer D454.6 (DO)
- net at D455.2 (CI): now also D456.5 (CO); no longer D454.5 (CO)
- net at D456.2 (CI): now also D457.5 (CO); no longer D455.5 (CO)
- net at D456.1 (DI): now also D457.6 (DO); no longer D455.6 (DO)
- net at D512.5 (CO): now also Q2 out1.2 (Pin_2)
- net at D512.6 (DO): now also Q2 out1.1 (Pin_1)
- net at D245.2 (CI): now also D292.5 (CO); no longer D244.5 (CO)
- net at D245.1 (DI): now also D292.6 (DO); no longer D244.6 (DO)
- net at D224.2 (CI): now also D262.5 (CO); no longer D223.5 (CO)
- net at D224.1 (DI): now also D262.6 (DO); no longer D223.6 (DO)
- net at D98.1 (DI): now also D146.6 (DO); no longer D97.6 (DO)
- net at D98.2 (CI): now also D146.5 (CO); no longer D97.5 (CO)
- net at D1.1 (DI): now also Q4 in1.1 (Pin_1)
- net at D1.2 (CI): now also Q4 in1.2 (Pin_2)
- net at D2.2 (CI): now also D3.5 (CO); no longer D1.5 (CO)
- net at D2.1 (DI): now also D3.6 (DO); no longer D1.6 (DO)
- net at D46.6 (DO): now also D7.1 (DI); no longer D47.1 (DI)
- net at D46.5 (CO): now also D7.2 (CI); no longer D47.2 (CI)
- net at D47.5 (CO): now also D6.2 (CI); no longer D48.2 (CI)
- net at D47.6 (DO): now also D6.1 (DI); no longer D48.1 (DI)
- net at D19.2 (CI): now also D34.5 (CO); no longer D18.5 (CO)
- net at D19.1 (DI): now also D34.6 (DO); no longer D18.6 (DO)
- net at D182.5 (CO): now also D163.2 (CI); no longer D183.2 (CI)
- net at D182.6 (DO): now also D163.1 (DI); no longer D183.1 (DI)
- net at D421.6 (DO): now also D420.1 (DI); no longer D422.1 (DI)
- net at D421.5 (CO): now also D420.2 (CI); no longer D422.2 (CI)
- net at D422.5 (CO): now also D421.2 (CI); no longer D423.2 (CI)
- net at D422.6 (DO): now also D421.1 (DI); no longer D423.1 (DI)
- net at D467.2 (CI): now also D468.5 (CO); no longer D466.5 (CO)
- net at D467.1 (DI): now also D468.6 (DO); no longer D466.6 (DO)
- net at D25.6 (DO): now also D464.1 (DI); no longer D26.1 (DI)
- net at D25.5 (CO): now also D464.2 (CI); no longer D26.2 (CI)
- net at D457.2 (CI): now also D458.5 (CO); no longer D456.5 (CO)
- net at D457.1 (DI): now also D458.6 (DO); no longer D456.6 (DO)
- net at D500.2 (CI): now also D501.5 (CO); no longer D499.5 (CO)
- net at D500.1 (DI): now also D501.6 (DO); no longer D499.6 (DO)
- net at D472.1 (DI): now also D473.6 (DO); no longer D471.6 (DO)
- net at D472.2 (CI): now also D473.5 (CO); no longer D471.5 (CO)
- net at D472.5 (CO): now also D471.2 (CI); no longer D473.2 (CI)
- net at D472.6 (DO): now also D471.1 (DI); no longer D473.1 (DI)
- net at D502.1 (DI): now also D503.6 (DO); no longer D501.6 (DO)
- net at D502.2 (CI): now also D503.5 (CO); no longer D501.5 (CO)
- net at D502.5 (CO): now also D501.2 (CI); no longer D503.2 (CI)
- net at D502.6 (DO): now also D501.1 (DI); no longer D503.1 (DI)
- net at D451.6 (DO): now also D426.1 (DI); no longer D452.1 (DI)
- net at D451.5 (CO): now also D426.2 (CI); no longer D452.2 (CI)
- net at D452.5 (CO): now also D425.2 (CI); no longer D453.2 (CI)
- net at D452.6 (DO): now also D425.1 (DI); no longer D453.1 (DI)
- net at D437.5 (CO): now also D396.2 (CI); no longer D438.2 (CI)
- net at D437.6 (DO): now also D396.1 (DI); no longer D438.1 (DI)
- net at D458.2 (CI): now also D459.5 (CO); no longer D457.5 (CO)
- net at D458.1 (DI): now also D459.6 (DO); no longer D457.6 (DO)
- net at D474.1 (DI): now also D475.6 (DO); no longer D473.6 (DO)
- net at D474.2 (CI): now also D475.5 (CO); no longer D473.5 (CO)
- net at D475.2 (CI): now also D476.5 (CO); no longer D474.5 (CO)
- net at D475.1 (DI): now also D476.6 (DO); no longer D474.6 (DO)
- net at D369.6 (DO): now also D368.1 (DI); no longer D370.1 (DI)
- net at D369.5 (CO): now also D368.2 (CI); no longer D370.2 (CI)
- net at D370.5 (CO): now also D369.2 (CI); no longer D371.2 (CI)
- net at D370.6 (DO): now also D369.1 (DI); no longer D371.1 (DI)
- net at D408.1 (DI): now also D409.6 (DO); no longer D407.6 (DO)
- net at D408.2 (CI): now also D409.5 (CO); no longer D407.5 (CO)
- net at D408.5 (CO): now also D371.2 (CI); no longer D409.2 (CI)
- net at D408.6 (DO): now also D371.1 (DI); no longer D409.1 (DI)
- net at D362.5 (CO): now also D319.2 (CI); no longer D363.2 (CI)
- net at D362.6 (DO): now also D319.1 (DI); no longer D363.1 (DI)
- net at D420.6 (DO): now also D419.1 (DI); no longer D421.1 (DI)
- net at D420.5 (CO): now also D419.2 (CI); no longer D421.2 (CI)
- net at D129.1 (DI): now also D128.6 (DO)
- net at D129.2 (CI): now also D128.5 (CO)
- net at D129.5 (CO): now also D119.2 (CI); no longer D130.2 (CI)
- net at D129.6 (DO): now also D119.1 (DI); no longer D130.1 (DI)
- net at D330.5 (CO): now also D308.2 (CI); no longer D331.2 (CI)
- net at D330.6 (DO): now also D308.1 (DI); no longer D331.1 (DI)
- net at D195.2 (CI): now also D147.5 (CO); no longer D194.5 (CO)
- net at D195.1 (DI): now also D147.6 (DO); no longer D194.6 (DO)
- net at D289.1 (DI): now also D295.6 (DO); no longer D288.6 (DO)
- net at D289.2 (CI): now also D295.5 (CO); no longer D288.5 (CO)
- net at D477.2 (CI): now also D478.5 (CO); no longer D476.5 (CO)
- net at D477.1 (DI): now also D478.6 (DO); no longer D476.6 (DO)
- net at D5.1 (DI): now also D6.6 (DO); no longer D4.6 (DO)
- net at D5.2 (CI): now also D6.5 (CO); no longer D4.5 (CO)
- net at D5.5 (CO): now also D4.2 (CI); no longer D6.2 (CI)
- net at D5.6 (DO): now also D4.1 (DI); no longer D6.1 (DI)
- net at D351.2 (CI): now also D383.5 (CO); no longer D350.5 (CO)
- net at D351.1 (DI): now also D383.6 (DO); no longer D350.6 (DO)
- net at D410.1 (DI): now also D411.6 (DO); no longer D409.6 (DO)
- net at D410.2 (CI): now also D411.5 (CO); no longer D409.5 (CO)
- net at D410.5 (CO): now also D409.2 (CI); no longer D411.2 (CI)
- net at D410.6 (DO): now also D409.1 (DI); no longer D411.1 (DI)
- net at D497.2 (CI): now also D498.5 (CO); no longer D496.5 (CO)
- net at D497.1 (DI): now also D498.6 (DO); no longer D496.6 (DO)
- net at D171.6 (DO): now also D123.1 (DI); no longer D172.1 (DI)
- net at D171.5 (CO): now also D123.2 (CI); no longer D172.2 (CI)
- net at D35.1 (DI): now also D61.6 (DO); no longer D34.6 (DO)
- net at D35.2 (CI): now also D61.5 (CO); no longer D34.5 (CO)
- net at D469.1 (DI): now also D470.6 (DO); no longer D468.6 (DO)
- net at D469.2 (CI): now also D470.5 (CO); no longer D468.5 (CO)
- net at D469.5 (CO): now also D468.2 (CI); no longer D470.2 (CI)
- net at D469.6 (DO): now also D468.1 (DI); no longer D470.1 (DI)
- net at D250.5 (CO): now also D236.2 (CI); no longer D251.2 (CI)
- net at D250.6 (DO): now also D236.1 (DI); no longer D251.1 (DI)
- net at D296.1 (DI): now also D341.6 (DO); no longer D295.6 (DO)
- net at D296.2 (CI): now also D341.5 (CO); no longer D295.5 (CO)
- net at D75.6 (DO): now also q3 out1.1 (Pin_1); no longer D76.1 (DI)
- net at D75.5 (CO): now also q3 out1.2 (Pin_2); no longer D76.2 (CI)
- net at D461.1 (DI): now also D462.6 (DO); no longer D460.6 (DO)
- net at D461.2 (CI): now also D462.5 (CO); no longer D460.5 (CO)
- net at D461.5 (CO): now also D460.2 (CI); no longer D462.2 (CI)
- net at D461.6 (DO): now also D460.1 (DI); no longer D462.1 (DI)
- net at D390.6 (DO): now also D342.1 (DI); no longer D391.1 (DI)
- net at D390.5 (CO): now also D342.2 (CI); no longer D391.2 (CI)
- net at D391.5 (CO): now also D439.2 (CI); no longer D392.2 (CI)
- net at D391.6 (DO): now also D439.1 (DI); no longer D392.1 (DI)
- net at D416.6 (DO): now also D415.1 (DI); no longer D417.1 (DI)
- net at D416.5 (CO): now also D415.2 (CI); no longer D417.2 (CI)
- net at D417.5 (CO): now also D416.2 (CI); no longer D418.2 (CI)
- net at D417.6 (DO): now also D416.1 (DI); no longer D418.1 (DI)
- net at D463.6 (DO): now also D462.1 (DI); no longer D464.1 (DI)
- net at D463.5 (CO): now also D462.2 (CI); no longer D464.2 (CI)
- net at D263.1 (DI): now also D277.6 (DO); no longer D262.6 (DO)
- net at D263.2 (CI): now also D277.5 (CO); no longer D262.5 (CO)
- net at D147.2 (CI): now also Q1 in1.2 (Pin_2); no longer D146.5 (CO)
- net at D147.1 (DI): now also Q1 in1.1 (Pin_1); no longer D146.6 (DO)
- net at D366.2 (CI): now also D367.5 (CO); no longer D365.5 (CO)
- net at D366.1 (DI): now also D367.6 (DO); no longer D365.6 (DO)
- net at D459.2 (CI): now also D460.5 (CO); no longer D458.5 (CO)
- net at D459.1 (DI): now also D460.6 (DO); no longer D458.6 (DO)
- net at D367.2 (CI): now also D368.5 (CO); no longer D366.5 (CO)
- net at D367.1 (DI): now also D368.6 (DO); no longer D366.6 (DO)
- net at D49.1 (DI): now also D1.6 (DO); no longer D48.6 (DO)
- net at D49.2 (CI): now also D1.5 (CO); no longer D48.5 (CO)
- net at D62.2 (CI): now also D87.5 (CO); no longer D61.5 (CO)
- net at D62.1 (DI): now also D87.6 (DO); no longer D61.6 (DO)
- net at D293.2 (CI): now also D196.5 (CO); no longer D292.5 (CO)
- net at D293.1 (DI): now also D196.6 (DO); no longer D292.6 (DO)
- net at D463.1 (DI): now also D467.6 (DO); no longer D462.6 (DO)
- net at D463.2 (CI): now also D467.5 (CO); no longer D462.5 (CO)
- net at D235.6 (DO): now also D207.1 (DI); no longer D236.1 (DI)
- net at D235.5 (CO): now also D207.2 (CI); no longer D236.2 (CI)
- net at D122.5 (CO): now also D74.2 (CI); no longer D123.2 (CI)
- net at D122.6 (DO): now also D74.1 (DI); no longer D123.1 (DI)
- net at D278.1 (DI): now also D307.6 (DO); no longer D277.6 (DO)
- net at D278.2 (CI): now also D307.5 (CO); no longer D277.5 (CO)
- net at D2.6 (DO): now also D488.1 (DI); no longer D3.1 (DI)
- net at D2.5 (CO): now also D488.2 (CI); no longer D3.2 (CI)
- net at D424.6 (DO): now also D423.1 (DI); no longer D425.1 (DI)
- net at D424.5 (CO): now also D423.2 (CI); no longer D425.2 (CI)
- net at D425.5 (CO): now also D424.2 (CI); no longer D426.2 (CI)
- net at D425.6 (DO): now also D424.1 (DI); no longer D426.1 (DI)
- net at D219.1 (DI): now also D223.6 (DO); no longer D218.6 (DO)
- net at D219.2 (CI): now also D223.5 (CO); no longer D218.5 (CO)
- net at D438.5 (CO): now also D392.2 (CI); no longer D439.2 (CI)
- net at D438.6 (DO): now also D392.1 (DI); no longer D439.1 (DI)
- net at D441.1 (DI): now also D487.6 (DO); no longer D440.6 (DO)
- net at D441.2 (CI): now also D487.5 (CO); no longer D440.5 (CO)
- net at D506.1 (DI): now also D507.6 (DO); no longer D505.6 (DO)
- net at D506.2 (CI): now also D507.5 (CO); no longer D505.5 (CO)
- net at D506.5 (CO): now also D505.2 (CI); no longer D507.2 (CI)
- net at D506.6 (DO): now also D505.1 (DI); no longer D507.1 (DI)
- net at D318.6 (DO): now also Q1 out1.1 (Pin_1); no longer D319.1 (DI)
- net at D318.5 (CO): now also Q1 out1.2 (Pin_2); no longer D319.2 (CI)
- net at D73.5 (CO): now also D26.2 (CI); no longer D74.2 (CI)
- net at D73.6 (DO): now also D26.1 (DI); no longer D74.1 (DI)
- net at D220.5 (CO): now also Q4 out1.2 (Pin_2); no longer D221.2 (CI)
- net at D220.6 (DO): now also Q4 out1.1 (Pin_1); no longer D221.1 (DI)
- net at D195.5 (CO): now also D148.2 (CI); no longer D196.2 (CI)
- net at D195.6 (DO): now also D148.1 (DI); no longer D196.1 (DI)
- net at D162.6 (DO): now also D130.1 (DI); no longer D163.1 (DI)
- net at D162.5 (CO): now also D130.2 (CI); no longer D163.2 (CI)
- net at D418.5 (CO): now also D417.2 (CI); no longer D419.2 (CI)
- net at D418.6 (DO): now also D417.1 (DI); no longer D419.1 (DI)
- net at D419.6 (DO): now also D418.1 (DI); no longer D420.1 (DI)
- net at D419.5 (CO): now also D418.2 (CI); no longer D420.2 (CI)
- net at D414.6 (DO): now also D413.1 (DI); no longer D415.1 (DI)
- net at D414.5 (CO): now also D413.2 (CI); no longer D415.2 (CI)
- net at D415.5 (CO): now also D414.2 (CI); no longer D416.2 (CI)
- net at D415.6 (DO): now also D414.1 (DI); no longer D416.1 (DI)
- net at D413.6 (DO): now also D412.1 (DI); no longer D414.1 (DI)
- net at D413.5 (CO): now also D412.2 (CI); no longer D414.2 (CI)
- net at D317.5 (CO): now also D269.2 (CI); no longer D318.2 (CI)
- net at D317.6 (DO): now also D269.1 (DI); no longer D318.1 (DI)
- net at D508.1 (DI): now also D466.6 (DO); no longer D507.6 (DO)
- net at D508.2 (CI): now also D466.5 (CO); no longer D507.5 (CO)
- net at D423.5 (CO): now also D422.2 (CI); no longer D424.2 (CI)
- net at D423.6 (DO): now also D422.1 (DI); no longer D424.1 (DI)
- net at D141.1 (DI): now also D150.6 (DO); no longer D140.6 (DO)
- net at D141.2 (CI): now also D150.5 (CO); no longer D140.5 (CO)
- net at D118.6 (DO): now also D76.1 (DI); no longer D119.1 (DI)
- net at D118.5 (CO): now also D76.2 (CI); no longer D119.2 (CI)
- net at D197.1 (DI): now also D244.6 (DO); no longer D196.6 (DO)
- net at D197.2 (CI): now also D244.5 (CO); no longer D196.5 (CO)
- net at D256.5 (CO): now also D257.2 (CI)
- net at D256.6 (DO): now also D257.1 (DI)
- net at D453.5 (CO): now also D452.2 (CI); no longer D454.2 (CI)
- net at D453.6 (DO): now also D452.1 (DI); no longer D454.1 (DI)
- net at D206.5 (CO): now also D183.2 (CI); no longer D207.2 (CI)
- net at D206.6 (DO): now also D183.1 (DI); no longer D207.1 (DI)
- net at D372.2 (CI): now also D407.5 (CO); no longer D371.5 (CO)
- net at D372.1 (DI): now also D407.6 (DO); no longer D371.6 (DO)
- net at D412.5 (CO): now also D411.2 (CI); no longer D413.2 (CI)
- net at D412.6 (DO): now also D411.1 (DI); no longer D413.1 (DI)
- net at D151.2 (CI): now also D194.5 (CO); no longer D150.5 (CO)
- net at D151.1 (DI): now also D194.6 (DO); no longer D150.6 (DO)
- net at D504.6 (DO): now also D503.1 (DI); no longer D505.1 (DI)
- net at D504.5 (CO): now also D503.2 (CI); no longer D505.2 (CI)
- net at D504.1 (DI): now also D505.6 (DO); no longer D503.6 (DO)
- net at D504.2 (CI): now also D505.5 (CO); no longer D503.5 (CO)
- net at D268.6 (DO): now also D221.1 (DI); no longer D269.1 (DI)
- net at D268.5 (CO): now also D221.2 (CI); no longer D269.2 (CI)
- new net: D391.1 (DI), Q3 in1.1 (Pin_1)
- new net: D391.2 (CI), Q3 in1.2 (Pin_2)
- new net: D18.6 (DO), D507.1 (DI)
- new net: D18.5 (CO), D507.2 (CI)
- new net: D365.2 (CI), D366.5 (CO)
- new net: D365.1 (DI), D366.6 (DO)
- new net: D331.1 (DI), D350.6 (DO)
- new net: D331.2 (CI), D350.5 (CO)
- new net: D364.2 (CI), D365.5 (CO)
- new net: D364.1 (DI), D365.6 (DO)
- new net: D251.2 (CI), D288.5 (CO)
- new net: D251.1 (DI), D288.6 (DO)
- new net: D172.2 (CI), D218.5 (CO)
- new net: D172.1 (DI), D218.6 (DO)
- new net: D454.1 (DI), D455.6 (DO)
- new net: D454.2 (CI), D455.5 (CO)
- new net: D453.2 (CI), D454.5 (CO)
- new net: D453.1 (DI), D454.6 (DO)
- new net: D107.2 (CI), D140.5 (CO)
- new net: D107.1 (DI), D140.6 (DO)
- new net: D370.2 (CI), D371.5 (CO)
- new net: D370.1 (DI), D371.6 (DO)
- new net: D196.1 (DI), Q2 in1.1 (Pin_1)
- new net: D196.2 (CI), Q2 in1.2 (Pin_2)
- new net: D48.2 (CI), D50.5 (CO)
- new net: D48.1 (DI), D50.6 (DO)
- new net: D3.2 (CI), D4.5 (CO)
- new net: D3.1 (DI), D4.6 (DO)
- new net: D438.2 (CI), D440.5 (CO)
- new net: D438.1 (DI), D440.6 (DO)
- new net: D47.1 (DI), D48.6 (DO)
- new net: D47.2 (CI), D48.5 (CO)
- new net: D470.2 (CI), D471.5 (CO)
- new net: D470.1 (DI), D471.6 (DO)
- new net: D478.2 (CI), D497.5 (CO)
- new net: D478.1 (DI), D497.6 (DO)
- new net: D473.1 (DI), D474.6 (DO)
- new net: D473.2 (CI), D474.5 (CO)
