File: pcb/core/core.kicad_pcb (KiCad board)
At the start: 2 copper layers, 73 x 101.5 mm, 10 parts, among them J1 MIC1, U1 Teensy4.0

Commit message: update
Parts:
- added REF**: MountingHole_3.2mm_M3_DIN965, MountingHole:MountingHole_3.2mm_M3_DIN965, F.Cu at (20.5, 21.5)
- added REF**: MountingHole_3.2mm_M3_DIN965, MountingHole:MountingHole_3.2mm_M3_DIN965, F.Cu at (80.0, 22.5)
- added REF**: MountingHole_3.2mm_M3_DIN965, MountingHole:MountingHole_3.2mm_M3_DIN965, F.Cu at (19.5, 112.5)
Other:
- board text added: "LOLLY-CORE"
